Commit message: added arm urdf file and PointCLoud2ToLaserScan repo for autonomy and arm control

File: install/my_bot/share/my_bot/description/depth_camera.xacro (robot description, xacro)
@@ -4,5 +4,5 @@
         <parent link="chassis"/>
         <child link="camera_link"/>
-        <origin xyz="0.205 0 0.28" rpy="0 0 0"/>
+        <origin xyz="0.208 0 0.28" rpy="0 0 0"/>
     </joint>
     <link name="camera_link">
@@ -11,5 +11,5 @@
                 <box size="0.010 0.03 0.03"/>
             </geometry>
-            <material name="red"/>
+            <material name="orange"/>
         </visual>
     </link>

File: install/my_bot/share/my_bot/description/macros.xacro (robot description, xacro)
@@ -1,4 +1,5 @@
 <?xml version="1.0"?>
 <robot xmlns:xacro="http://www.ros.org/wiki/xacro"  >
+    <!-- <xacro:include filename="robot_core.xacro"/> -->
     <!--ROS2_CONTROL MACROS-->
     <!--Joint Creator-->
@@ -100,3 +101,30 @@
         </inertial>
     </xacro:macro>
+    <!--Arm Inertial Macros-->
+    <xacro:property name="intom" value="0.0254"/>
+	<xacro:property name="lbtokg" value="0.454"/>
+	<xacro:property name="lbsqintokgsqm" value="703.07"/>
+    <xacro:macro name="sw_origin" params="x y z roll:=0 pitch:=0 yaw:=0">
+        <origin xyz="${x*intom} ${-z*intom} ${y*intom}" rpy="${roll} ${pitch} ${yaw}"/>
+    </xacro:macro>
+    <xacro:macro name="sw_visual" params="file">
+        <visual>
+            <origin xyz="0 0 0" rpy="${radians(90)} 0 0"/>
+            <geometry>
+                <mesh filename="package://my_bot/description/mesh/${file}.STL"/>
+            </geometry>
+            <material name="white"/>
+        </visual>
+    </xacro:macro>
+    <!-- Units: lb, in, lb*in^2 -->
+    <xacro:macro name="sw_inertial" params="m X Y Z Lxx Lxy Lxz Lyy Lyz Lzz">
+        <inertial>
+            <mass value="${m*lbtokg}"/>
+            <xacro:sw_origin x="${X}" y="${Y}" z="${Z}"/>
+            <inertia
+                ixx="${Lxx*lbsqintokgsqm}" ixy="${Lxz*lbsqintokgsqm}" ixz="${-Lxy*lbsqintokgsqm}"
+                iyy="${Lzz*lbsqintokgsqm}" iyz="${-Lyz*lbsqintokgsqm}"
+                izz="${Lyy*lbsqintokgsqm}"/>
+        </inertial>
+    </xacro:macro>
 </robot>

File: install/my_bot/share/my_bot/description/robot.urdf.xacro (robot description, xacro)
@@ -1,7 +1,8 @@
 <?xml version="1.0"?>
 <robot xmlns:xacro="http://www.ros.org/wiki/xacro"  name="robot">
-    <xacro:include filename="robot_core.xacro"/>
-    <xacro:include filename="ros2_control.xacro"/>
+    <!-- <xacro:include filename="robot_core.xacro"/>
+    <xacro:include filename="ros2_control.xacro"/> -->
+    <xacro:include filename="arm.xacro"/>
     <!-- <xacro:include filename="camera.xacro"/> -->
-    <xacro:include filename="depth_camera.xacro"/>
+    <!-- <xacro:include filename="depth_camera.xacro"/> -->
 </robot>

File: install/my_bot/share/my_bot/description/robot_core.xacro (robot description, xacro)
@@ -1,5 +1,5 @@
 <?xml version="1.0"?>
 <robot xmlns:xacro="http://www.ros.org/wiki/xacro"  >
-     <xacro:include filename="macros.xacro"/>
+    <xacro:include filename="macros.xacro"/>
     <!-- Declaring Constants -->
     <xacro:property name="wheel_radius" value="0.05" />
@@ -7,5 +7,5 @@
     <xacro:property name="chassis_origin" value="0 0 0.1" />
     <!-- <xacro:include filename="inertial_macros.xacro"/> -->
-    <material name="white">
+    <!-- <material name="white">
         <color rgba="1 1 1 1"/>
     </material>
@@ -18,5 +18,5 @@
     <material name="black">
         <color rgba="0 0 0 1"/>
-    </material>
+    </material> -->
     <!-- WHEELS -->
     <!--With Encoders-->
@@ -30,4 +30,12 @@
     <!--BASE LINK-->
     <link name="base_link">
+    </link>
+    <!--BASE_FOOTPRINT LINK-->
+    <joint name ="base_footprint_joint" type="fixed">
+        <parent link="base_link"/>
+        <child link="base_footprint"/>
+        <origin xyz ="0 0 0" rpy="0 0 0"/>
+    </joint>
+    <link name ="base_footprint">
     </link>
     <!--CHASSIS LINK-->
@@ -60,3 +68,36 @@
         <mu2 value="0.001"/>
     </gazebo>
+    <!--IMU Sensor-->
+    <link name="imu">
+        <sensor name="my_imu" type="imu">
+            <always_on>true</always_on>
+            <!--Publish at 30 hz-->
+            <update_rate>30</update_rate>
+            <plugin name="my_imu_plugin" filename="libgazebo_ros_imu_sensor.so">
+                <ros>
+                    <!--Will publish to /imu/data-->
+                    <namespace>/imu</namespace>
+                    <remapping>~/out:=data</remapping>
+                </ros>
+                <!--frame_name ommited, will be "my_link"-->
+            </plugin>
+        </sensor>
+    </link>
+    <link name ="imu_sensor">
+    </link>
+    <gazebo reference="imu_sensor">
+        <sensor name="my_imu" type="imu">
+            <always_on>true</always_on>
+            <!--Publish at 30 hz-->
+            <update_rate>30</update_rate>
+            <plugin name="my_imu_plugin" filename="libgazebo_ros_imu_sensor.so">
+                <ros>
+                    <!--Will publish to /imu/data-->
+                    <namespace>/imu</namespace>
+                    <remapping>~/out:=data</remapping>
+                </ros>
+                <!--frame_name ommited, will be "my_link"-->
+            </plugin>
+        </sensor>
+    </gazebo>
 </robot>
