Commit message: Fixed code to simulate arm and control through a GUI

File: install/my_bot/share/my_bot/description/arm.urdf.xacro (robot description, xacro)
@@ -14,10 +14,4 @@
         <color rgba="0 0 0 1"/>
     </material>
-	<link name="base_link">
-	</link>
-	<joint name="dummy_joint" type="fixed">
-     <parent link="base_link"/>
-     <child link="arm_a1"/>
-   </joint>
 	<link name="arm_a1">
 		<xacro:sw_visual file="ARM-A01"/>
@@ -37,5 +31,5 @@
 	<joint name="arm_j1" type="revolute">
 		<xacro:sw_origin x="-3.50000000" y="0.51712500" z="0"/>
-		<parent link="base_link"/>
+		<parent link="arm_a1"/>
 		<child link="arm_a2" />
 		<axis xyz="0 0 1"/>

File: install/my_bot/share/my_bot/description/macros.xacro (robot description, xacro)
@@ -112,5 +112,5 @@
             <origin xyz="0 0 0" rpy="${radians(90)} 0 0"/>
             <geometry>
-                <mesh filename="package://my_bot/description/mesh/${file}.STL"/>
+                <mesh filename="file://$(find my_bot)/description/mesh/${file}.STL"/>
             </geometry>
             <material name="white"/>

Commit message: added arm gazebo simulation and ros2 controllers

File: install/my_bot/share/my_bot/description/arm.urdf.xacro (robot description, xacro)
@@ -2,5 +2,5 @@
 <robot xmlns:xacro="http://www.ros.org/wiki/xacro" name="robot_arm" >
 	<xacro:include filename="macros.xacro"/>
-	 <material name="white">
+	<material name="white">
         <color rgba="1 1 1 1"/>
     </material>
@@ -14,4 +14,9 @@
         <color rgba="0 0 0 1"/>
     </material>
+	<!--Dummy Link-->
+	<!-- <link name="world">
+	</link> -->
+	<!--Arm Links-->
+	<!--Arm 1-->
 	<link name="arm_a1">
 		<xacro:sw_visual file="ARM-A01"/>
@@ -27,4 +32,5 @@
 			Lyz="-0.00376"
 			Lzz="69.49319"
+			file="ARM-A01"
 		/>
 	</link>
@@ -36,4 +42,9 @@
 		<limit lower="${radians(-180)}" upper="${radians(180)}" effort="40" velocity="30"/>
 	</joint>
+	<!-- <joint name="dummy_joint" type="fixed">
+		<parent link="dummy"/>
+		<child link="arm_a1"/>
+	</joint> -->
+	<!--Arm 2-->
 	<link name="arm_a2">
 		<xacro:sw_visual file="ARM-A02"/>
@@ -49,4 +60,5 @@
 			Lyz="0.14287"
 			Lzz="14.594"
+			file="ARM-A02"
 		/>
 	</link>
@@ -58,4 +70,5 @@
 		<limit lower="${radians(-135)}" upper="${radians(15)}" effort="125" velocity="30"/>
 	</joint>
+	<!--Arm 3-->
 	<link name="arm_a3">
 		<xacro:sw_visual file="ARM-A03"/>
@@ -71,4 +84,5 @@
 			Lyz="-0.00494"
 			Lzz="465.43"
+			file="ARM-A03"
 		/>
 	</link>
@@ -80,4 +94,5 @@
 		<limit lower="${radians(-120)}" upper="${radians(120)}" effort="80" velocity="30"/>
 	</joint>
+	<!--Arm 4-->
 	<link name="arm_a4">
 		<xacro:sw_visual file="ARM-A04"/>
@@ -93,4 +108,5 @@
 			Lyz="-0.0001"
 			Lzz="227.3199"
+			file="ARM-A04"
 		/>
 	</link>
@@ -102,4 +118,5 @@
 		<limit effort="30" velocity="30"/>
 	</joint>
+	<!--Arm 5-->
 	<link name="arm_a5">
 		<xacro:sw_visual file="ARM-A05"/>
@@ -115,4 +132,5 @@
 			Lyz="-0.0010"
 			Lzz="30.6708"
+			file="ARM-A05"
 		/>
 	</link>
@@ -124,4 +142,5 @@
 		<limit lower="${radians(-90)}" upper="${radians(90)}" effort="30" velocity="30"/>
 	</joint>
+	<!--Arm 6-->
 	<link name="arm_a6">
 		<xacro:sw_visual file="ARM-A06"/>
@@ -137,4 +156,5 @@
 			Lyz="0.0008"
 			Lzz="6.2503"
+			file="ARM-A06"
 		/>
 	</link>
@@ -146,17 +166,37 @@
 		<limit effort="30" velocity="30"/>
 	</joint>
+	<!--Arm 7-->
 	<link name="arm_a7">
-		<xacro:sw_inertial
-			m="1"
-			X="0"
-			Y="0"
-			Z="0"
-			Lxx="0.01"
-			Lxy="0.00"
-			Lxz="0.00"
-			Lyy="0.01"
-			Lyz="0.00"
-			Lzz="0.01"
-		/>
-	</link>
+		<inertial>
+            <mass value="${lbtokg}"/>
+            <xacro:sw_origin x="0" y="0" z="0"/>
+            <inertia
+                ixx="${0.01*lbsqintokgsqm}" ixy="${0.00*lbsqintokgsqm}" ixz="${-0.00*lbsqintokgsqm}"
+                iyy="${0.01*lbsqintokgsqm}" iyz="${-0.00*lbsqintokgsqm}"
+                izz="${0.01*lbsqintokgsqm}"/>
+        </inertial>
+        <collision>
+            <xacro:sw_origin x="0" y="0" z="0"/>
+            <geometry>
+                <box size="0.01 0.01 0.01"/>
+            </geometry>
+        </collision>
+	</link>
+	<!--Defining ROS2 Control Joints-->
+	<ros2_control name="GazeboSystem" type="system">
+        <hardware>
+        	<plugin>gazebo_ros2_control/GazeboSystem</plugin>
+        </hardware>
+		<xacro:arm_joint_creator name="arm_j1"/>
+		<xacro:arm_joint_creator name="arm_j2"/>
+		<xacro:arm_joint_creator name="arm_j3"/>
+		<xacro:arm_joint_creator name="arm_j4"/>
+        <xacro:arm_joint_creator name="arm_j5"/>
+		<xacro:arm_joint_creator name="arm_j6"/>
+	</ros2_control>
+	<gazebo>
+        <plugin name="gazebo_ros2_control" filename="libgazebo_ros2_control.so">
+            <parameters> $(find my_bot)/config/arm_controllers.yaml</parameters>
+        </plugin>
+    </gazebo>
 </robot>

File: src/my_bot/description/arm.urdf.xacro (robot description, xacro)
@@ -15,6 +15,6 @@
     </material>
 	<!--Dummy Link-->
-	<link name="dummy">
-	</link>
+	<!-- <link name="world">
+	</link> -->
 	<!--Arm Links-->
 	<!--Arm 1-->
@@ -42,8 +42,8 @@
 		<limit lower="${radians(-180)}" upper="${radians(180)}" effort="40" velocity="30"/>
 	</joint>
-	<joint name="dummy_joint" type="fixed">
+	<!-- <joint name="dummy_joint" type="fixed">
 		<parent link="dummy"/>
 		<child link="arm_a1"/>
-	</joint>
+	</joint> -->
 	<!--Arm 2-->
 	<link name="arm_a2">
@@ -161,6 +161,6 @@
 	<joint name="arm_j6" type="continuous">
 		<xacro:sw_origin x="2.98622047" y="0" z="0"/>
-		<parent link="arm_a5"/>
-		<child link="arm_a6"/>
+		<parent link="arm_a6"/>
+		<child link="arm_a7"/>
 		<axis xyz="1 0 0"/>
 		<limit effort="30" velocity="30"/>

Commit message: testing

File: install/my_bot/share/my_bot/description/arm.urdf.xacro (robot description, xacro)
@@ -15,8 +15,15 @@
     </material>
 	<!--Dummy Link-->
-	<!-- <link name="world">
-	</link> -->
+	<link name="world">
+	</link>
 	<!--Arm Links-->
 	<!--Arm 1-->
+	<joint name="arm_j1" type="revolute">
+		<xacro:sw_origin x="-3.50000000" y="0.51712500" z="0"/>
+		<parent link="arm_a1"/>
+		<child link="arm_a2" />
+		<axis xyz="0 0 1"/>
+		<limit lower="${radians(-180)}" upper="${radians(180)}" effort="40" velocity="30"/>
+	</joint>
 	<link name="arm_a1">
 		<xacro:sw_visual file="ARM-A01"/>
@@ -35,15 +42,9 @@
 		/>
 	</link>
-	<joint name="arm_j1" type="revolute">
-		<xacro:sw_origin x="-3.50000000" y="0.51712500" z="0"/>
-		<parent link="arm_a1"/>
-		<child link="arm_a2" />
-		<axis xyz="0 0 1"/>
-		<limit lower="${radians(-180)}" upper="${radians(180)}" effort="40" velocity="30"/>
-	</joint>
-	<!-- <joint name="dummy_joint" type="fixed">
-		<parent link="dummy"/>
+	<joint name="dummy_joint" type="fixed">
+		<origin xyz="0 0 0"/>
+		<parent link="world"/>
 		<child link="arm_a1"/>
-	</joint> -->
+	</joint>
 	<!--Arm 2-->
 	<link name="arm_a2">
