Commit message: rviz working wiht moveit and model

File: install/my_bot/share/my_bot/description/arm.urdf (robot description, URDF)
Before this commit: robot robot_arm, 7 links, 6 joints
Links:
- added link base_link
Joints:
- added joint dummy_joint: type fixed, parent base_link, child arm_a1
- joint arm_j1: limit lower=-3.141592653589793 upper=3.141592653589793 effort=40 velocity=30 -> lower=-3.141592653589793 upper=3.141592653589793 effort=40.0 velocity=30.0
- joint arm_j2: limit lower=-2.356194490192345 upper=0.2617993877991494 effort=125 velocity=30 -> lower=-2.356194490192345 upper=0.2617993877991494 effort=125.0 velocity=30.0
- joint arm_j3: limit lower=-2.0943951023931953 upper=2.0943951023931953 effort=80 velocity=30 -> lower=-2.0943951023931953 upper=2.0943951023931953 effort=80.0 velocity=30.0
- joint arm_j4: limit effort=30 velocity=30 -> effort=30.0 velocity=30.0
- joint arm_j5: limit lower=-1.5707963267948966 upper=1.5707963267948966 effort=30 velocity=30 -> lower=-1.5707963267948966 upper=1.5707963267948966 effort=30.0 velocity=30.0
- joint arm_j6: limit effort=30 velocity=30 -> effort=30.0 velocity=30.0

File: install/my_bot/share/my_bot/description/arm.urdf.xacro (robot description, xacro)
@@ -15,15 +15,11 @@
     </material>
 	<!--Dummy Link-->
-	<link name="world">
-	</link>
+	<link name="base_link"/>
+	<joint name="dummy_joint" type="fixed">
+		<parent link="base_link"/>
+		<child link="arm_a1"/>
+	</joint>
 	<!--Arm Links-->
 	<!--Arm 1-->
-	<joint name="arm_j1" type="revolute">
-		<xacro:sw_origin x="-3.50000000" y="0.51712500" z="0"/>
-		<parent link="arm_a1"/>
-		<child link="arm_a2" />
-		<axis xyz="0 0 1"/>
-		<limit lower="${radians(-180)}" upper="${radians(180)}" effort="40" velocity="30"/>
-	</joint>
 	<link name="arm_a1">
 		<xacro:sw_visual file="ARM-A01"/>
@@ -42,8 +38,10 @@
 		/>
 	</link>
-	<joint name="dummy_joint" type="fixed">
-		<origin xyz="0 0 0"/>
-		<parent link="world"/>
-		<child link="arm_a1"/>
+	<joint name="arm_j1" type="revolute">
+		<xacro:sw_origin x="-3.50000000" y="0.51712500" z="0"/>
+		<parent link="arm_a1"/>
+		<child link="arm_a2" />
+		<axis xyz="0 0 1"/>
+		<limit lower="${radians(-180)}" upper="${radians(180)}" effort="40.0" velocity="30.0"/>
 	</joint>
 	<!--Arm 2-->
@@ -69,5 +67,5 @@
 		<child link="arm_a3"/>
 		<axis xyz="0 1 0"/>
-		<limit lower="${radians(-135)}" upper="${radians(15)}" effort="125" velocity="30"/>
+		<limit lower="${radians(-135)}" upper="${radians(15)}" effort="125.0" velocity="30.0"/>
 	</joint>
 	<!--Arm 3-->
@@ -93,5 +91,5 @@
 		<child link="arm_a4"/>
 		<axis xyz="0 1 0"/>
-		<limit lower="${radians(-120)}" upper="${radians(120)}" effort="80" velocity="30"/>
+		<limit lower="${radians(-120)}" upper="${radians(120)}" effort="80.0" velocity="30.0"/>
 	</joint>
 	<!--Arm 4-->
@@ -117,5 +115,5 @@
 		<child link="arm_a5"/>
 		<axis xyz="1 0 0"/>
-		<limit effort="30" velocity="30"/>
+		<limit effort="30.0" velocity="30.0"/>
 	</joint>
 	<!--Arm 5-->
@@ -141,5 +139,5 @@
 		<child link="arm_a6"/>
 		<axis xyz="0 1 0"/>
-		<limit lower="${radians(-90)}" upper="${radians(90)}" effort="30" velocity="30"/>
+		<limit lower="${radians(-90)}" upper="${radians(90)}" effort="30.0" velocity="30.0"/>
 	</joint>
 	<!--Arm 6-->
@@ -165,5 +163,5 @@
 		<child link="arm_a7"/>
 		<axis xyz="1 0 0"/>
-		<limit effort="30" velocity="30"/>
+		<limit effort="30.0" velocity="30.0"/>
 	</joint>
 	<!--Arm 7-->
@@ -187,5 +185,5 @@
 	<ros2_control name="GazeboSystem" type="system">
         <hardware>
-        	<plugin>gazebo_ros2_control/GazeboSystem</plugin>
+        	<plugin>mock_components/GenericSystem</plugin>
         </hardware>
 		<xacro:arm_joint_creator name="arm_j1"/>

File: install/my_bot/share/my_bot/description/macros.xacro (robot description, xacro)
@@ -15,13 +15,9 @@
     <xacro:macro name="arm_joint_creator" params="name">
             <joint name="${name}">
-                <command_interface name="effort">
-                    <param name="min">-10000</param>
-                    <param name="min">10000</param>
-                </command_interface>
+                <command_interface name="position"/>
                 <state_interface name="position">
                     <param name="initial_value">0.0</param>
                 </state_interface>
                 <state_interface name="velocity"/>
-                <state_interface name="effort"/>
             </joint>
     </xacro:macro>
