Commit message: pid changed to avoid moveit

File: install/my_bot/share/my_bot/description/arm_gazebo.urdf.xacro (robot description, xacro)
@@ -192,5 +192,5 @@
   	</link>
 	<!--Defining ROS2 Control Joints-->
-	<ros2_control name="GazeboSystem" type="system">
+	<!-- <ros2_control name="GazeboSystem" type="system">
         <hardware>
         	<plugin>gazebo_ros2_control/GazeboSystem</plugin>
@@ -202,28 +202,20 @@
         <xacro:arm_joint_creator name="arm_j5"/>
 		<xacro:arm_joint_creator name="arm_j6"/>
-	</ros2_control>
-	<!-- <ros2_control name="yurs_motor" type="actuator">
+	</ros2_control> -->
+	<ros2_control name="yurs_motor" type="actuator">
 		<hardware>
 			<plugin>yurs_hardware/yurs_motor</plugin>
 			<param name="can_interface">can0</param>
 		</hardware>
-		<joint name="front_left_wheel_joint">
-			<param name="device_id">0</param>
-			<param name="counts_per_rev">1512</param>
-		</joint>
-		<joint name="front_right_wheel_joint">
-			<param name="device_id">3</param>
-			<param name="counts_per_rev">1512</param>
-		</joint>
-		<joint name="middle_left_wheel_joint">
-			<param name="device_id">1</param>
-			<param name="counts_per_rev">1512</param>
-		</joint>
-		<joint name="middle_right_wheel_joint">
-			<param name="device_id">4</param>
-			<param name="counts_per_rev">1512</param>
-		</joint>
-		<joint name="rear_left_wheel_joint">
-			<param name="device_id">2</param>
+ 		<joint name="arm_j1">
+			<param name="device_id">6</param>
+			<param name="counts_per_rev">1512</param>
+		</joint>
+		<joint name="arm_j2">
+			<param name="device_id">7</param>
+			<param name="counts_per_rev">1512</param>
+		</joint>
+		<joint name="arm_j3">
+			<param name="device_id">8</param>
 			<param name="counts_per_rev">1512</param>
 		</joint>
@@ -232,10 +224,17 @@
 			<param name="counts_per_rev">1512</param>
 		</joint>
+		<joint name="arm_j5">
+			<param name="device_id">10</param>
+			<param name="counts_per_rev">1512</param>
+		</joint>
+		<joint name="arm_j6">
+			<param name="device_id">11</param>
+			<param name="counts_per_rev">1512</param>
+		</joint>
 	</ros2_control>
- -->
-	<gazebo>
+	<!-- <gazebo>
         <plugin name="gazebo_ros2_control" filename="libgazebo_ros2_control.so">
             <parameters> $(find my_bot)/config/arm_gazebo_controllers.yaml</parameters>
         </plugin>
-    </gazebo>
+    </gazebo> -->
 </robot>

Commit message: working arm with really bad PID values

File: install/my_bot/share/my_bot/description/arm_gazebo.urdf.xacro (robot description, xacro)
@@ -14,10 +14,9 @@
         <color rgba="0 0 0 1"/>
     </material>
-	<!--Dummy Link-->
-	<link name="base_link"/>
-	<joint name="dummy_joint" type="fixed">
-		<parent link="base_link"/>
-		<child link="arm_a1"/>
-	</joint>
+	 <link name="world"/>
+        <joint name="fix" type="fixed">
+            <parent link="world"/>
+            <child link="arm_a1"/>
+        </joint>
 	<!--Arm Links-->
 	<!--Arm 1-->

File: install/my_bot/share/my_bot/description/arm_hardware.urdf.xacro (robot description, xacro)
@@ -17,4 +17,5 @@
 	<link name="base_link"/>
 	<joint name="dummy_joint" type="fixed">
+		<origin xyz="0 1-0 0" rpy="0 0 0"/>
 		<parent link="base_link"/>
 		<child link="arm_a1"/>
@@ -231,25 +232,25 @@
  		<joint name="arm_j1">
 			<param name="device_id">6</param>
-			<param name="counts_per_rev">1512</param>
+			<param name="counts_per_rev">1050</param>
 		</joint>
 		<joint name="arm_j2">
 			<param name="device_id">7</param>
-			<param name="counts_per_rev">1512</param>
+			<param name="counts_per_rev">5250</param>
 		</joint>
 		<joint name="arm_j3">
 			<param name="device_id">8</param>
-			<param name="counts_per_rev">1512</param>
+			<param name="counts_per_rev">5250</param>
 		</joint>
 		<joint name="arm_j4">
 			<param name="device_id">9</param>
-			<param name="counts_per_rev">1512</param>
+			<param name="counts_per_rev">1149.1597</param>
 		</joint>
 		<joint name="arm_j5">
 			<param name="device_id">10</param>
-			<param name="counts_per_rev">1512</param>
+			<param name="counts_per_rev">1149.1597</param>
 		</joint>
 		<joint name="arm_j6">
 			<param name="device_id">11</param>
-			<param name="counts_per_rev">1512</param>
+			<param name="counts_per_rev">1149.1597</param>
 		</joint>
 		<!-- <joint name="arm_j7">

File: install/my_bot/share/my_bot/description/macros.xacro (robot description, xacro)
@@ -163,4 +163,5 @@
                     izz="${Lyy*lbsqintokgsqm}"/>
             </inertial>
+<!--
             <collision>
                 <origin rpy="${radians(90)} 0 0" xyz="0 0 0"/>
@@ -168,5 +169,5 @@
                     <mesh filename="file://$(find my_bot)/description/mesh/${file}.STL" />
                 </geometry>
-            </collision>
+            </collision> -->
         </link>
         <joint name="arm_j${component_number}" type="${type}">
