Commit message: MOVEIt group runs

File: install/arm_control_moveit_config/share/arm_control_moveit_config/config/arm.urdf (robot description, URDF)
Before this commit: robot robot_arm, 8 links, 7 joints
Joints:
- joint arm_j1: limit lower=-3.141592653589793 upper=3.141592653589793 effort=40 velocity=30 -> lower=-3.141592653589793 upper=3.141592653589793 effort=40.0 velocity=30.0
- joint arm_j2: limit lower=-2.356194490192345 upper=0.2617993877991494 effort=125 velocity=30 -> lower=-2.356194490192345 upper=0.2617993877991494 effort=125.0 velocity=30.0
- joint arm_j3: limit lower=-2.0943951023931953 upper=2.0943951023931953 effort=80 velocity=30 -> lower=-2.0943951023931953 upper=2.0943951023931953 effort=80.0 velocity=30.0
- joint arm_j4: limit effort=30 velocity=30 -> effort=30.0 velocity=30.0
- joint arm_j5: limit lower=-1.5707963267948966 upper=1.5707963267948966 effort=30 velocity=30 -> lower=-1.5707963267948966 upper=1.5707963267948966 effort=30.0 velocity=30.0
- joint arm_j6: limit effort=30 velocity=30 -> effort=30.0 velocity=30.0

File: install/arm_control_moveit_config/share/arm_control_moveit_config/config/arm.urdf.xacro (robot description, xacro)
@@ -196,5 +196,5 @@
 	<gazebo>
         <plugin name="gazebo_ros2_control" filename="libgazebo_ros2_control.so">
-            <parameters> $(find my_bot)/config/arm_controllers.yaml</parameters>
+            <parameters> $(find arm_control_moveit_config)/config/ros2_controllers.yaml</parameters>
         </plugin>
     </gazebo>
