Commit message: PID WORKS, Gazebo unable to handle Float32

File: install/arm_control_moveit_config/share/arm_control_moveit_config/config/robot_arm.ros2_control.xacro (robot description, xacro)
@@ -13,5 +13,5 @@
                   <param name="initial_value">${initial_positions['arm_j5']}</param>
                 </state_interface>
-                <state_interface name="velocity"/>
+                <!-- <state_interface name="velocity"/> -->
             </joint>
             <joint name="arm_j6">
@@ -20,5 +20,5 @@
                   <param name="initial_value">${initial_positions['arm_j6']}</param>
                 </state_interface>
-                <state_interface name="velocity"/>
+                <!-- <state_interface name="velocity"/> -->
             </joint>
             <joint name="arm_j1">
@@ -27,5 +27,5 @@
                   <param name="initial_value">${initial_positions['arm_j1']}</param>
                 </state_interface>
-                <state_interface name="velocity"/>
+                <!-- <state_interface name="velocity"/> -->
             </joint>
             <joint name="arm_j2">
@@ -34,5 +34,5 @@
                   <param name="initial_value">${initial_positions['arm_j2']}</param>
                 </state_interface>
-                <state_interface name="velocity"/>
+                <!-- <state_interface name="velocity"/> -->
             </joint>
             <joint name="arm_j3">
@@ -41,5 +41,5 @@
                   <param name="initial_value">${initial_positions['arm_j3']}</param>
                 </state_interface>
-                <state_interface name="velocity"/>
+                <!-- <state_interface name="velocity"/> -->
             </joint>
             <joint name="arm_j4">
@@ -48,5 +48,5 @@
                   <param name="initial_value">${initial_positions['arm_j4']}</param>
                 </state_interface>
-                <state_interface name="velocity"/>
+                <!-- <state_interface name="velocity"/> -->
             </joint>
         </ros2_control>

File: install/arm_control_moveit_config/share/arm_control_moveit_config/config/robot_arm.urdf.xacro (robot description, xacro)
@@ -6,4 +6,4 @@
     <!-- Import control_xacro -->
     <xacro:include filename="robot_arm.ros2_control.xacro" />
-    <xacro:robot_arm_ros2_control name="FakeSystem" initial_positions_file="$(arg initial_positions_file)"/>
+    <xacro:robot_arm_ros2_control name="GazeboSystem" initial_positions_file="$(arg initial_positions_file)"/>
 </robot>

File: install/my_bot/share/my_bot/description/arm_gazebo.urdf.xacro (robot description, xacro)
@@ -191,6 +191,27 @@
 		</collision>
   	</link>
+	<!-- <joint name="arm_j7" type="prismatic">
+            <origin xyz="0 0 0" rpy="0 0 0"/>
+            <parent link="arm_a7"/>
+            <child link="arm_a8"/>
+            <axis xyz="1 0 0"/>
+			 <limit effort="50" lower="-50" upper="50" velocity="50"/>
+	</joint> -->
+	<!-- <link name="arm_a8">
+		<inertial>
+			<mass value="0.454"/>
+			<origin rpy="0 0 0" xyz="0.0 0.0 0.0"/>
+			<inertia ixx="7.0307" ixy="0.0" ixz="-0.0" iyy="7.0307" iyz="-0.0" izz="7.0307"/>
+		</inertial>
+		<collision>
+		<origin rpy="0 0 0" xyz="0.0 0.0 0.0"/>
+		<geometry>
+			<box size="0.01 0.01 0.01"/>
+		</geometry>
+		</collision>
+  	</link>
+ -->
 	<!--Defining ROS2 Control Joints-->
-	<!-- <ros2_control name="GazeboSystem" type="system">
+	<ros2_control name="GazeboSystem" type="system">
         <hardware>
         	<plugin>gazebo_ros2_control/GazeboSystem</plugin>
@@ -202,6 +223,6 @@
         <xacro:arm_joint_creator name="arm_j5"/>
 		<xacro:arm_joint_creator name="arm_j6"/>
-	</ros2_control> -->
-	<ros2_control name="yurs_motor" type="actuator">
+	</ros2_control>
+	<!-- <ros2_control name="yurs_motor" type="actuator">
 		<hardware>
 			<plugin>yurs_hardware/yurs_motor</plugin>
@@ -232,9 +253,13 @@
 			<param name="counts_per_rev">1512</param>
 		</joint>
-	</ros2_control>
-	<!-- <gazebo>
+		<joint name="arm_j7">
+			<param name="device_id">12</param>
+			<param name="counts_per_rev">1512</param>
+		</joint>
+	</ros2_control> -->
+	<gazebo>
         <plugin name="gazebo_ros2_control" filename="libgazebo_ros2_control.so">
             <parameters> $(find my_bot)/config/arm_gazebo_controllers.yaml</parameters>
         </plugin>
-    </gazebo> -->
+    </gazebo>
 </robot>

Commit message: IT WORKKKKKSSS

File: install/arm_control_moveit_config/share/arm_control_moveit_config/config/robot_arm.ros2_control.xacro (robot description, xacro)
@@ -3,52 +3,38 @@
     <xacro:macro name="robot_arm_ros2_control" params="name initial_positions_file">
         <xacro:property name="initial_positions" value="${load_yaml(initial_positions_file)['initial_positions']}"/>
-        <ros2_control name="${name}" type="system">
-            <hardware>
-                <!-- By default, set up controllers for simulation. This won't work on real hardware -->
-                <plugin>mock_components/GenericSystem</plugin>
-            </hardware>
-            <joint name="arm_j5">
-                <command_interface name="effort"/>
-                <state_interface name="position">
-                  <param name="initial_value">${initial_positions['arm_j5']}</param>
-                </state_interface>
-                <!-- <state_interface name="velocity"/> -->
-            </joint>
-            <joint name="arm_j6">
-                <command_interface name="effort"/>
-                <state_interface name="position">
-                  <param name="initial_value">${initial_positions['arm_j6']}</param>
-                </state_interface>
-                <!-- <state_interface name="velocity"/> -->
-            </joint>
-            <joint name="arm_j1">
-                <command_interface name="effort"/>
-                <state_interface name="position">
-                  <param name="initial_value">${initial_positions['arm_j1']}</param>
-                </state_interface>
-                <!-- <state_interface name="velocity"/> -->
-            </joint>
-            <joint name="arm_j2">
-                <command_interface name="effort"/>
-                <state_interface name="position">
-                  <param name="initial_value">${initial_positions['arm_j2']}</param>
-                </state_interface>
-                <!-- <state_interface name="velocity"/> -->
-            </joint>
-            <joint name="arm_j3">
-                <command_interface name="effort"/>
-                <state_interface name="position">
-                  <param name="initial_value">${initial_positions['arm_j3']}</param>
-                </state_interface>
-                <!-- <state_interface name="velocity"/> -->
-            </joint>
-            <joint name="arm_j4">
-                <command_interface name="effort"/>
-                <state_interface name="position">
-                  <param name="initial_value">${initial_positions['arm_j4']}</param>
-                </state_interface>
-                <!-- <state_interface name="velocity"/> -->
-            </joint>
-        </ros2_control>
+       <ros2_control name="yurs_motor" type="actuator">
+        <hardware>
+          <plugin>yurs_hardware/yurs_motor</plugin>
+          <param name="can_interface">can0</param>
+        </hardware>
+        <joint name="arm_j1">
+          <param name="device_id">6</param>
+          <param name="counts_per_rev">1512</param>
+        </joint>
+        <joint name="arm_j2">
+          <param name="device_id">7</param>
+          <param name="counts_per_rev">1512</param>
+        </joint>
+        <joint name="arm_j3">
+          <param name="device_id">8</param>
+          <param name="counts_per_rev">1512</param>
+        </joint>
+        <joint name="arm_j4">
+          <param name="device_id">9</param>
+          <param name="counts_per_rev">1512</param>
+        </joint>
+        <joint name="arm_j5">
+          <param name="device_id">10</param>
+          <param name="counts_per_rev">1512</param>
+        </joint>
+        <joint name="arm_j6">
+          <param name="device_id">11</param>
+          <param name="counts_per_rev">1512</param>
+        </joint>
+        <!-- <joint name="arm_j7">
+          <param name="device_id">12</param>
+          <param name="counts_per_rev">1512</param>
+        </joint> -->
+	</ros2_control>
     </xacro:macro>
 </robot>

File: install/my_bot/share/my_bot/description/arm_hardware.urdf.xacro (robot description, xacro)
@@ -253,8 +253,8 @@
 			<param name="counts_per_rev">1512</param>
 		</joint>
-		<joint name="arm_j7">
+		<!-- <joint name="arm_j7">
 			<param name="device_id">12</param>
 			<param name="counts_per_rev">1512</param>
-		</joint>
+		</joint> -->
 	</ros2_control>
 	<!-- <gazebo>

Commit message: pid controll

File: install/arm_control_moveit_config/share/arm_control_moveit_config/config/robot_arm.ros2_control.xacro (robot description, xacro)
@@ -3,5 +3,52 @@
     <xacro:macro name="robot_arm_ros2_control" params="name initial_positions_file">
         <xacro:property name="initial_positions" value="${load_yaml(initial_positions_file)['initial_positions']}"/>
-       <ros2_control name="yurs_motor" type="actuator">
+  <ros2_control name="GazeboSystem" type="system">
+    <hardware>
+      <plugin>gazebo_ros2_control/GazeboSystem</plugin>
+    </hardware>
+    <joint name="arm_j1">
+      <command_interface name="effort"/>
+      <!-- <state_interface name="position">
+        <param name="initial_value">180</param>
+      </state_interface> -->
+      <!-- <state_interface name="velocity"/> -->
+    </joint>
+    <joint name="arm_j2">
+      <command_interface name="effort"/>
+      <!-- <state_interface name="position">
+        <param name="initial_value">-1</param>
+      </state_interface> -->
+      <!-- <state_interface name="velocity"/> -->
+    </joint>
+    <joint name="arm_j3">
+      <command_interface name="effort"/>
+      <!-- <state_interface name="position">
+        <param name="initial_value">-120</param>
+      </state_interface> -->
+      <!-- <state_interface name="velocity"/> -->
+    </joint>
+    <joint name="arm_j4">
+      <command_interface name="effort"/>
+      <!-- <state_interface name="position">
+        <param name="initial_value">1</param>
+      </state_interface> -->
+      <!-- <state_interface name="velocity"/> -->
+    </joint>
+    <joint name="arm_j5">
+      <command_interface name="effort"/>
+      <!-- <state_interface name="position">
+        <param name="initial_value">-11</param>
+      </state_interface> -->
+      <!-- <state_interface name="velocity"/> -->
+    </joint>
+    <joint name="arm_j6">
+      <command_interface name="effort"/>
+      <!-- <state_interface name="position">
+        <param name="initial_value">3</param>
+      </state_interface> -->
+      <!-- <state_interface name="velocity"/> -->
+    </joint>
+  </ros2_control>
+       <!-- <ros2_control name="yurs_motor" type="actuator">
         <hardware>
           <plugin>yurs_hardware/yurs_motor</plugin>
@@ -32,9 +79,9 @@
           <param name="counts_per_rev">1512</param>
         </joint>
-        <!-- <joint name="arm_j7">
+        <joint name="arm_j7">
           <param name="device_id">12</param>
           <param name="counts_per_rev">1512</param>
-        </joint> -->
-	</ros2_control>
+        </joint>
+	</ros2_control> -->
     </xacro:macro>
 </robot>
