Commit message: working Effort and velocity PID for simultion with tunning and cli pubishers

File: src/arm_control_moveit_config/config/arm_gazebo.urdf.xacro (robot description, xacro)
@@ -14,11 +14,9 @@
         <color rgba="0 0 0 1"/>
     </material>
-	<!--Dummy Link-->
-	<link name="base_link"/>
-	<joint name="dummy_joint" type="fixed">
-		<origin xyz="0 0 0" rpy="0 0 0"/>
-		<parent link="base_link"/>
-		<child link="arm_a1"/>
-	</joint>
+	 <link name="world"/>
+        <joint name="fix" type="fixed">
+            <parent link="world"/>
+            <child link="arm_a1"/>
+        </joint>
 	<!--Arm Links-->
 	<!--Arm 1-->
@@ -46,5 +44,5 @@
 		joint_X = "-3.50000000"
 		joint_Y = "0.51712500"
-		joint_Z = "0.0"
+		joint_Z = "0"
 	/>
 	<!--Arm 2-->
@@ -57,6 +55,6 @@
 		axis = "0 1 0"
 		Lxx="21.53"
-		Lxy="0.0"
-		Lxz="0.0"
+		Lxy="0"
+		Lxz="0"
 		Lyy="10.896"
 		Lyz="0.14287"
@@ -70,7 +68,7 @@
 		upper_limit = "${radians(15)}"
 		velocity_limit = "300000.0"
-		joint_X = "0.0"
+		joint_X = "0"
 		joint_Y = "3.75000000"
-		joint_Z = "0.0"
+		joint_Z = "0"
 	/>
 	<!--Arm 3-->
@@ -97,6 +95,6 @@
 		velocity_limit = "300000.0"
 		joint_X = "18.00000000"
-		joint_Y = "0.0"
-		joint_Z = "0.0"
+		joint_Y = "0"
+		joint_Z = "0"
 	/>
 	<!--Arm 4-->
@@ -123,6 +121,6 @@
 		velocity_limit = "300000.0"
 		joint_X = "4.48622047"
-		joint_Y = "0.0"
-		joint_Z = "0.0"
+		joint_Y = "0"
+		joint_Z = "0"
 	/>
 	<!--Arm 5-->
@@ -131,5 +129,5 @@
 		type = "revolute"
 		parent_link = "arm_a5"
-		child_link = "arm_a6"
+		child_link = "arm_a7"
 		mass="2.8972"
 		axis = "0 1 0"
@@ -149,9 +147,9 @@
 		velocity_limit = "300000.0"
 		joint_X = "17.25000000"
-		joint_Y = "0.0"
-		joint_Z = "0.0"
+		joint_Y = "0"
+		joint_Z = "0"
 	/>
 	<!--Arm 6-->
-	<xacro:arm_component
+	<!-- <xacro:arm_component
 		component_number ="6"
 		type = "revolute"
@@ -175,7 +173,7 @@
 		velocity_limit = "300000.0"
 		joint_X = "2.98622047"
-		joint_Y = "0.0"
-		joint_Z = "0.0"
-	/>
+		joint_Y = "0"
+		joint_Z = "0"
+	/> -->
 	<!--Arm 7-->
 	<link name="arm_a7">
@@ -214,37 +212,19 @@
  -->
 	<!--Defining ROS2 Control Joints-->
-	<ros2_control name="yurs_motor" type="actuator">
-		<hardware>
-			<plugin>yurs_hardware/yurs_motor</plugin>
-			<param name="can_interface">can0</param>
-		</hardware>
- 		<joint name="arm_j1">
-			<param name="device_id">6</param>
-			<param name="counts_per_rev">1050</param>
-		</joint>
-		<joint name="arm_j2">
-			<param name="device_id">7</param>
-			<param name="counts_per_rev">5250</param>
-		</joint>
-		<joint name="arm_j3">
-			<param name="device_id">8</param>
-			<param name="counts_per_rev">5250</param>
-		</joint>
-		<joint name="arm_j4">
-			<param name="device_id">9</param>
-			<param name="counts_per_rev">1149.1597</param>
-		</joint>
-		<joint name="arm_j5">
-			<param name="device_id">10</param>
-			<param name="counts_per_rev">1149.1597</param>
-		</joint>
-		<joint name="arm_j6">
-			<param name="device_id">11</param>
-			<param name="counts_per_rev">1149.1597</param>
-		</joint>
-		<!-- <joint name="arm_j7">
-			<param name="device_id">12</param>
-			<param name="counts_per_rev">1512</param>
-		</joint> -->
+	<ros2_control name="GazeboSystem" type="system">
+        <hardware>
+        	<plugin>gazebo_ros2_control/GazeboSystem</plugin>
+        </hardware>
+		<xacro:arm_joint_creator name="arm_j1"/>
+		<xacro:arm_joint_creator name="arm_j2"/>
+		<xacro:arm_joint_creator name="arm_j3"/>
+		<xacro:arm_joint_creator name="arm_j4"/>
+        <xacro:arm_joint_creator name="arm_j5"/>
+		<!-- <xacro:arm_joint_creator name="arm_j6"/>	 -->
 	</ros2_control>
+	<gazebo>
+        <plugin name="gazebo_ros2_control" filename="libgazebo_ros2_control.so">
+            <parameters> $(find my_bot)/config/arm_gazebo_controllers.yaml</parameters>
+        </plugin>
+    </gazebo>
 </robot>

File: src/arm_control_moveit_config/config/robot_arm.ros2_control.xacro (robot description, xacro)
@@ -3,54 +3,47 @@
     <xacro:macro name="robot_arm_ros2_control" params="name initial_positions_file">
         <xacro:property name="initial_positions" value="${load_yaml(initial_positions_file)['initial_positions']}"/>
-<!---->
-  <!-- <ros2_control name="GazeboSystem" type="system">
+  <ros2_control name="GazeboSystem" type="system">
     <hardware>
       <plugin>gazebo_ros2_control/GazeboSystem</plugin>
     </hardware>
     <joint name="arm_j1">
-      <command_interface name="effort"/> -->
-      <!-- <state_interface name="position">
+      <command_interface name="effort"/>
+      <state_interface name="position">
         <param name="initial_value">180</param>
-      </state_interface> -->
-      <!-- <state_interface name="velocity"/> -->
-    <!-- </joint>
+      </state_interface>
+    </joint>
     <joint name="arm_j2">
-      <command_interface name="effort"/> -->
-      <!-- <state_interface name="position">
+      <command_interface name="effort"/>
+      <state_interface name="position">
         <param name="initial_value">-1</param>
-      </state_interface> -->
-      <!-- <state_interface name="velocity"/> -->
-    <!-- </joint>
+      </state_interface>
+    </joint>
     <joint name="arm_j3">
-      <command_interface name="effort"/> -->
-      <!-- <state_interface name="position">
+      <command_interface name="effort"/>
+      <state_interface name="position">
         <param name="initial_value">-120</param>
-      </state_interface> -->
-      <!-- <state_interface name="velocity"/> -->
-    <!-- </joint>
+      </state_interface>
+    </joint>
     <joint name="arm_j4">
-      <command_interface name="effort"/> -->
-      <!-- <state_interface name="position">
+      <command_interface name="effort"/>
+      <state_interface name="position">
         <param name="initial_value">1</param>
-      </state_interface> -->
-      <!-- <state_interface name="velocity"/> -->
-    <!-- </joint>
+      </state_interface>
+    </joint>
     <joint name="arm_j5">
-      <command_interface name="effort"/> -->
-      <!-- <state_interface name="position">
+      <command_interface name="effort"/>
+      <state_interface name="position">
         <param name="initial_value">-11</param>
-      </state_interface> -->
-      <!-- <state_interface name="velocity"/> -->
-    <!-- </joint>
+      </state_interface>
+    </joint>
     <joint name="arm_j6">
-      <command_interface name="effort"/> -->
-      <!-- <state_interface name="position">
+      <command_interface name="effort"/>
+      <state_interface name="position">
         <param name="initial_value">3</param>
-      </state_interface> -->
-      <!-- <state_interface name="velocity"/> -->
-    <!-- </joint>
-  </ros2_control> -->
-  <ros2_control name="yurs_motor" type="actuator">
-        <hardware>
+      </state_interface>
+    </joint>
+  </ros2_control>
+  <!-- <ros2_control name="yurs_motor" type="actuator"> -->
+        <!-- <hardware>
           <plugin>yurs_hardware/yurs_motor</plugin>
           <param name="can_interface">can0</param>
@@ -79,10 +72,10 @@
           <param name="device_id">11</param>
           <param name="counts_per_rev">1512</param>
-        </joint>
+        </joint> -->
         <!-- <joint name="arm_j7">
           <param name="device_id">12</param>
           <param name="counts_per_rev">1512</param>
         </joint> -->
-	</ros2_control>
+	<!-- </ros2_control> -->
     </xacro:macro>
 </robot>

File: src/my_bot/description/arm_gazebo.urdf.xacro (robot description, xacro)
@@ -223,38 +223,4 @@
 		<xacro:arm_joint_creator name="arm_j6"/>
 	</ros2_control>
-	<!-- <ros2_control name="yurs_motor" type="actuator">
-		<hardware>
-			<plugin>yurs_hardware/yurs_motor</plugin>
-			<param name="can_interface">can0</param>
-		</hardware>
- 		<joint name="arm_j1">
-			<param name="device_id">6</param>
-			<param name="counts_per_rev">1512</param>
-		</joint>
-		<joint name="arm_j2">
-			<param name="device_id">7</param>
-			<param name="counts_per_rev">1512</param>
-		</joint>
-		<joint name="arm_j3">
-			<param name="device_id">8</param>
-			<param name="counts_per_rev">1512</param>
-		</joint>
-		<joint name="arm_j4">
-			<param name="device_id">9</param>
-			<param name="counts_per_rev">1512</param>
-		</joint>
-		<joint name="arm_j5">
-			<param name="device_id">10</param>
-			<param name="counts_per_rev">1512</param>
-		</joint>
-		<joint name="arm_j6">
-			<param name="device_id">11</param>
-			<param name="counts_per_rev">1512</param>
-		</joint>
-		<joint name="arm_j7">
-			<param name="device_id">12</param>
-			<param name="counts_per_rev">1512</param>
-		</joint>
-	</ros2_control> -->
 	<gazebo>
         <plugin name="gazebo_ros2_control" filename="libgazebo_ros2_control.so">
