Commit message: controller

File: src/arm_control_moveit_config/config/robot_arm.ros2_control.xacro (robot description, xacro)
@@ -8,4 +8,11 @@
                 <plugin>mock_components/GenericSystem</plugin>
             </hardware>
+            <joint name="arm_j5">
+                <command_interface name="position"/>
+                <state_interface name="position">
+                  <param name="initial_value">${initial_positions['arm_j5']}</param>
+                </state_interface>
+                <state_interface name="velocity"/>
+            </joint>
             <joint name="arm_j6">
                 <command_interface name="position"/>
@@ -43,11 +50,4 @@
                 <state_interface name="velocity"/>
             </joint>
-            <joint name="arm_j5">
-                <command_interface name="position"/>
-                <state_interface name="position">
-                  <param name="initial_value">${initial_positions['arm_j5']}</param>
-                </state_interface>
-                <state_interface name="velocity"/>
-            </joint>
         </ros2_control>
     </xacro:macro>

File: src/my_bot/description/arm.urdf (robot description, URDF)
Before this commit: robot robot_arm, 8 links, 7 joints
Links:
- link arm_a1: mass 1.733599 -> 3.8185
- link arm_a2: mass 1.6581896 -> 3.6524
- link arm_a3: mass 2.9794204 -> 6.5626
- link arm_a4: mass 2.398936 -> 5.284
- link arm_a5: mass 1.3153288 -> 2.8972
- link arm_a6: mass 1.023543 -> 2.2545
Joints:
- joint arm_j4: limit effort=30.0 velocity=30.0 -> lower=-3.141592653589793 upper=3.141592653589793 effort=30.0 velocity=30.0
- joint arm_j6: limit effort=30.0 velocity=30.0 -> lower=-1.5707963267948966 upper=1.5707963267948966 effort=30.0 velocity=30.0; type continuous -> revolute

File: src/my_bot/description/arm.urdf.xacro (robot description, xacro)
@@ -22,164 +22,173 @@
 	<!--Arm Links-->
 	<!--Arm 1-->
-	<link name="arm_a1">
-		<xacro:sw_visual file="ARM-A01"/>
-		<xacro:sw_inertial
-			m="3.8185"
-			X="-3.34872"
-			Y="-7.71683"
-			Z="0.00031"
-			Lxx="100.85864"
-			Lxy="2.33423"
-			Lxz="-0.07753"
-			Lyy="40.30078"
-			Lyz="-0.00376"
-			Lzz="69.49319"
-			file="ARM-A01"
-		/>
-	</link>
-	<joint name="arm_j1" type="revolute">
-		<xacro:sw_origin x="-3.50000000" y="0.51712500" z="0"/>
-		<parent link="arm_a1"/>
-		<child link="arm_a2" />
-		<axis xyz="0 0 1"/>
-		<limit lower="${radians(-180)}" upper="${radians(180)}" effort="40.0" velocity="30.0"/>
-	</joint>
+	<xacro:arm_component
+		component_number ="1"
+		type = "revolute"
+		parent_link = "arm_a1"
+		child_link = "arm_a2"
+		mass = "3.8185"
+		axis = "0 0 1"
+		Lxx="100.85864"
+		Lxy="2.33423"
+		Lxz="-0.07753"
+		Lyy="40.30078"
+		Lyz="-0.00376"
+		Lzz="69.49319"
+		file="ARM-A01"
+		inertiaX = "-3.34872"
+		inertiaY = "-7.71683"
+		inertiaZ = "0.00031"
+		effort_limit = "40.0"
+		lower_limit = "${radians(-180)}"
+		upper_limit = "${radians(180)}"
+		velocity_limit = "30.0"
+		joint_X = "-3.50000000"
+		joint_Y = "0.51712500"
+		joint_Z = "0"
+	/>
 	<!--Arm 2-->
-	<link name="arm_a2">
-		<xacro:sw_visual file="ARM-A02"/>
-		<xacro:sw_inertial
-			m="3.6524"
-			X="0"
-			Y="2.7203"
-			Z="0.03799"
-			Lxx="21.53"
-			Lxy="0"
-			Lxz="0"
-			Lyy="10.896"
-			Lyz="0.14287"
-			Lzz="14.594"
-			file="ARM-A02"
-		/>
-	</link>
-	<joint name="arm_j2" type="revolute">
-		<xacro:sw_origin x="0" y="3.75000000" z="0"/>
-		<parent link="arm_a2"/>
-		<child link="arm_a3"/>
-		<axis xyz="0 1 0"/>
-		<limit lower="${radians(-135)}" upper="${radians(15)}" effort="125.0" velocity="30.0"/>
-	</joint>
+	<xacro:arm_component
+		component_number ="2"
+		type = "revolute"
+		parent_link = "arm_a2"
+		child_link = "arm_a3"
+		mass="3.6524"
+		axis = "0 1 0"
+		Lxx="21.53"
+		Lxy="0"
+		Lxz="0"
+		Lyy="10.896"
+		Lyz="0.14287"
+		Lzz="14.594"
+		file="ARM-A02"
+		inertiaX = "0"
+		inertiaY = "2.7203"
+		inertiaZ = "0.03799"
+		effort_limit = "125.0"
+		lower_limit = "${radians(-135)}"
+		upper_limit = "${radians(15)}"
+		velocity_limit = "30.0"
+		joint_X = "0"
+		joint_Y = "3.75000000"
+		joint_Z = "0"
+	/>
 	<!--Arm 3-->
-	<link name="arm_a3">
-		<xacro:sw_visual file="ARM-A03"/>
-		<xacro:sw_inertial
-			m="6.5626"
-			X="9.0018"
-			Y="-0.00037"
-			Z="4.4146"
-			Lxx="65.558"
-			Lxy="-0.15469"
-			Lxz="0.02472"
-			Lyy="525.31"
-			Lyz="-0.00494"
-			Lzz="465.43"
-			file="ARM-A03"
-		/>
-	</link>
-	<joint name="arm_j3" type="revolute">
-		<xacro:sw_origin x="18.00000000" y="0" z="0"/>
-		<parent link="arm_a3"/>
-		<child link="arm_a4"/>
-		<axis xyz="0 1 0"/>
-		<limit lower="${radians(-120)}" upper="${radians(120)}" effort="80.0" velocity="30.0"/>
-	</joint>
+	<xacro:arm_component
+		component_number ="3"
+		type = "revolute"
+		parent_link = "arm_a3"
+		child_link = "arm_a4"
+		mass="6.5626"
+		axis = "0 1 0"
+		Lxx="65.558"
+		Lxy="-0.15469"
+		Lxz="0.02472"
+		Lyy="525.31"
+		Lyz="-0.00494"
+		Lzz="465.43"
+		file="ARM-A03"
+		inertiaX="9.0018"
+		inertiaY="-0.00037"
+		inertiaZ="4.4146"
+		effort_limit = "80.0"
+		lower_limit = "${radians(-120)}"
+		upper_limit = "${radians(120)}"
+		velocity_limit = "30.0"
+		joint_X = "18.00000000"
+		joint_Y = "0"
+		joint_Z = "0"
+	/>
 	<!--Arm 4-->
-	<link name="arm_a4">
-		<xacro:sw_visual file="ARM-A04"/>
-		<xacro:sw_inertial
-			m="5.2840"
-			X="4.9938"
-			Y="0.0000"
-			Z="0.0189"
-			Lxx="17.7636"
-			Lxy="-0.0006"
-			Lxz="-1.1308"
-			Lyy="240.1392"
-			Lyz="-0.0001"
-			Lzz="227.3199"
-			file="ARM-A04"
-		/>
-	</link>
-	<joint name="arm_j4" type="continuous">
-		<xacro:sw_origin x="4.48622047" y="0" z="0"/>
-		<parent link="arm_a4"/>
-		<child link="arm_a5"/>
-		<axis xyz="1 0 0"/>
-		<limit effort="30.0" velocity="30.0"/>
-	</joint>
+	<xacro:arm_component
+		component_number ="4"
+		type = "continuous"
+		parent_link = "arm_a4"
+		child_link = "arm_a5"
+		mass="5.2840"
+		axis = "1 0 0"
+		Lxx="17.7636"
+		Lxy="-0.0006"
+		Lxz="-1.1308"
+		Lyy="240.1392"
+		Lyz="-0.0001"
+		Lzz="227.3199"
+		file="ARM-A04"
+		inertiaX="4.9938"
+		inertiaY="0.0000"
+		inertiaZ="0.0189"
+		effort_limit = "30.0"
+		lower_limit = "${radians(-180)}"
+		upper_limit = "${radians(180)}"
+		velocity_limit = "30.0"
+		joint_X = "4.48622047"
+		joint_Y = "0"
+		joint_Z = "0"
+	/>
 	<!--Arm 5-->
-	<link name="arm_a5">
-		<xacro:sw_visual file="ARM-A05"/>
-		<xacro:sw_inertial
-			m="2.8972"
-			X="14.8203"
-			Y="0.0000"
-			Z="0.2634"
-			Lxx="19.6638"
-			Lxy="-0.0018"
-			Lxz="1.7653"
-			Lyy="43.6205"
-			Lyz="-0.0010"
-			Lzz="30.6708"
-			file="ARM-A05"
-		/>
-	</link>
-	<joint name="arm_j5" type="revolute">
-		<xacro:sw_origin x="17.25000000" y="0" z="0"/>
-		<parent link="arm_a5"/>
-		<child link="arm_a6"/>
-		<axis xyz="0 1 0"/>
-		<limit lower="${radians(-90)}" upper="${radians(90)}" effort="30.0" velocity="30.0"/>
-	</joint>
+	<xacro:arm_component
+		component_number ="5"
+		type = "revolute"
+		parent_link = "arm_a5"
+		child_link = "arm_a6"
+		mass="2.8972"
+		axis = "0 1 0"
+		Lxx="19.6638"
+		Lxy="-0.0018"
+		Lxz="1.7653"
+		Lyy="43.6205"
+		Lyz="-0.0010"
+		Lzz="30.6708"
+		file="ARM-A05"
+		inertiaX="14.8203"
+		inertiaY="0.0000"
+		inertiaZ="0.2634"
+		effort_limit = "30.0"
+		lower_limit = "${radians(-90)}"
+		upper_limit = "${radians(90)}"
+		velocity_limit = "30.0"
+		joint_X = "17.25000000"
+		joint_Y = "0"
+		joint_Z = "0"
+	/>
 	<!--Arm 6-->
-	<link name="arm_a6">
-		<xacro:sw_visual file="ARM-A06"/>
-		<xacro:sw_inertial
-			m="2.2545"
-			X="1.6113"
-			Y="-0.0138"
-			Z="0.0240"
-			Lxx="8.2279"
-			Lxy="-0.0415"
-			Lxz="-0.0881"
-			Lyy="9.0021"
-			Lyz="0.0008"
-			Lzz="6.2503"
-			file="ARM-A06"
-		/>
-	</link>
-	<joint name="arm_j6" type="continuous">
-		<xacro:sw_origin x="2.98622047" y="0" z="0"/>
-		<parent link="arm_a6"/>
-		<child link="arm_a7"/>
-		<axis xyz="1 0 0"/>
-		<limit effort="30.0" velocity="30.0"/>
-	</joint>
+	<xacro:arm_component
+		component_number ="6"
+		type = "revolute"
+		parent_link = "arm_a6"
+		child_link = "arm_a7"
+		mass="2.2545"
+		axis = "1 0 0"
+		Lxx="8.2279"
+		Lxy="-0.0415"
+		Lxz="-0.0881"
+		Lyy="9.0021"
+		Lyz="0.0008"
+		Lzz="6.2503"
+		file="ARM-A06"
+		inertiaX="1.6113"
+		inertiaY="-0.0138"
+		inertiaZ="0.0240"
+		effort_limit = "30.0"
+		lower_limit = "${radians(-90)}"
+		upper_limit = "${radians(90)}"
+		velocity_limit = "30.0"
+		joint_X = "2.98622047"
+		joint_Y = "0"
+		joint_Z = "0"
+	/>
 	<!--Arm 7-->
 	<link name="arm_a7">
 		<inertial>
-            <mass value="${lbtokg}"/>
-            <xacro:sw_origin x="0" y="0" z="0"/>
-            <inertia
-                ixx="${0.01*lbsqintokgsqm}" ixy="${0.00*lbsqintokgsqm}" ixz="${-0.00*lbsqintokgsqm}"
-                iyy="${0.01*lbsqintokgsqm}" iyz="${-0.00*lbsqintokgsqm}"
-                izz="${0.01*lbsqintokgsqm}"/>
-        </inertial>
-        <collision>
-            <xacro:sw_origin x="0" y="0" z="0"/>
-            <geometry>
-                <box size="0.01 0.01 0.01"/>
-            </geometry>
-        </collision>
-	</link>
+		<mass value="0.454"/>
+		<origin rpy="0 0 0" xyz="0.0 0.0 0.0"/>
+		<inertia ixx="7.0307" ixy="0.0" ixz="-0.0" iyy="7.0307" iyz="-0.0" izz="7.0307"/>
+		</inertial>
+		<collision>
+		<origin rpy="0 0 0" xyz="0.0 0.0 0.0"/>
+		<geometry>
+			<box size="0.01 0.01 0.01"/>
+		</geometry>
+		</collision>
+  	</link>
 	<!--Defining ROS2 Control Joints-->
 	<ros2_control name="GazeboSystem" type="system">

File: src/my_bot/description/macros.xacro (robot description, xacro)
@@ -142,3 +142,39 @@
         </collision>
     </xacro:macro>
+    <!--DEFINING MY OWN MACROS CUZ WHOEVER DID THE ARM IS STUPID-->
+    <xacro:macro name="sw_origin" params="x y z roll:=0 pitch:=0 yaw:=0">
+        <origin xyz="${x*intom} ${-z*intom} ${y*intom}" rpy="${roll} ${pitch} ${yaw}"/>
+    </xacro:macro>
+    <xacro:macro name="arm_component" params=" component_number type parent_link child_link mass axis Lxx Lxy Lxz Lyy Lyz Lzz file inertiaX inertiaY inertiaZ effort_limit lower_limit upper_limit velocity_limit joint_X joint_Y joint_Z">
+        <link name="arm_a${component_number}">
+            <visual>
+                <origin rpy="${radians(90)} 0 0" xyz="0 0 0"/>
+                <geometry>
+                    <mesh filename="file://$(find my_bot)/description/mesh/${file}.STL" />
+                </geometry>
+                <material name="white"/>
+            </visual>
+            <inertial>
+                <mass value="${mass}"/>
+                <origin xyz="${inertiaX*intom} ${-inertiaZ*intom} ${inertiaY*intom}" rpy="0 0 0"/>
+                <inertia
+                    ixx="${Lxx*lbsqintokgsqm}" ixy="${Lxz*lbsqintokgsqm}" ixz="${-Lxy*lbsqintokgsqm}"
+                    iyy="${Lzz*lbsqintokgsqm}" iyz="${-Lyz*lbsqintokgsqm}"
+                    izz="${Lyy*lbsqintokgsqm}"/>
+            </inertial>
+            <collision>
+                <origin rpy="${radians(90)} 0 0" xyz="0 0 0"/>
+                <geometry>
+                    <mesh filename="file://$(find my_bot)/description/mesh/${file}.STL" />
+                </geometry>
+            </collision>
+        </link>
+        <joint name="arm_j${component_number}" type="${type}">
+            <origin xyz="${joint_X*intom} ${-joint_Z*intom} ${joint_Y*intom}" rpy="0 0 0"/>
+            <parent link="${parent_link}"/>
+            <child link="${child_link}"/>
+            <axis xyz="${axis}"/>
+            <limit effort="${effort_limit}" lower="${lower_limit}" upper="${upper_limit}" velocity="${velocity_limit}"/>
+        </joint>
+    </xacro:macro>
 </robot>

Commit message: fixed some bugs by testing on real hardware, PID yet to be calibrated.

File: src/arm_control_moveit_config/config/robot_arm.ros2_control.xacro (robot description, xacro)
@@ -3,52 +3,53 @@
     <xacro:macro name="robot_arm_ros2_control" params="name initial_positions_file">
         <xacro:property name="initial_positions" value="${load_yaml(initial_positions_file)['initial_positions']}"/>
-  <ros2_control name="GazeboSystem" type="system">
+<!---->
+  <!-- <ros2_control name="GazeboSystem" type="system">
     <hardware>
       <plugin>gazebo_ros2_control/GazeboSystem</plugin>
     </hardware>
     <joint name="arm_j1">
-      <command_interface name="effort"/>
+      <command_interface name="effort"/> -->
       <!-- <state_interface name="position">
         <param name="initial_value">180</param>
       </state_interface> -->
       <!-- <state_interface name="velocity"/> -->
-    </joint>
+    <!-- </joint>
     <joint name="arm_j2">
-      <command_interface name="effort"/>
+      <command_interface name="effort"/> -->
       <!-- <state_interface name="position">
         <param name="initial_value">-1</param>
       </state_interface> -->
       <!-- <state_interface name="velocity"/> -->
-    </joint>
+    <!-- </joint>
     <joint name="arm_j3">
-      <command_interface name="effort"/>
+      <command_interface name="effort"/> -->
       <!-- <state_interface name="position">
         <param name="initial_value">-120</param>
       </state_interface> -->
       <!-- <state_interface name="velocity"/> -->
-    </joint>
+    <!-- </joint>
     <joint name="arm_j4">
-      <command_interface name="effort"/>
+      <command_interface name="effort"/> -->
       <!-- <state_interface name="position">
         <param name="initial_value">1</param>
       </state_interface> -->
       <!-- <state_interface name="velocity"/> -->
-    </joint>
+    <!-- </joint>
     <joint name="arm_j5">
-      <command_interface name="effort"/>
+      <command_interface name="effort"/> -->
       <!-- <state_interface name="position">
         <param name="initial_value">-11</param>
       </state_interface> -->
       <!-- <state_interface name="velocity"/> -->
-    </joint>
+    <!-- </joint>
     <joint name="arm_j6">
-      <command_interface name="effort"/>
+      <command_interface name="effort"/> -->
       <!-- <state_interface name="position">
         <param name="initial_value">3</param>
       </state_interface> -->
       <!-- <state_interface name="velocity"/> -->
-    </joint>
-  </ros2_control>
-       <!-- <ros2_control name="yurs_motor" type="actuator">
+    <!-- </joint>
+  </ros2_control> -->
+  <ros2_control name="yurs_motor" type="actuator">
         <hardware>
           <plugin>yurs_hardware/yurs_motor</plugin>
@@ -79,9 +80,9 @@
           <param name="counts_per_rev">1512</param>
         </joint>
-        <joint name="arm_j7">
+        <!-- <joint name="arm_j7">
           <param name="device_id">12</param>
           <param name="counts_per_rev">1512</param>
-        </joint>
-	</ros2_control> -->
+        </joint> -->
+	</ros2_control>
     </xacro:macro>
 </robot>

File: src/my_bot/description/arm_hardware.urdf.xacro (robot description, xacro)
@@ -17,5 +17,5 @@
 	<link name="base_link"/>
 	<joint name="dummy_joint" type="fixed">
-		<origin xyz="0 1-0 0" rpy="0 0 0"/>
+		<origin xyz="0 0 0" rpy="0 0 0"/>
 		<parent link="base_link"/>
 		<child link="arm_a1"/>
@@ -46,5 +46,5 @@
 		joint_X = "-3.50000000"
 		joint_Y = "0.51712500"
-		joint_Z = "0"
+		joint_Z = "0.0"
 	/>
 	<!--Arm 2-->
@@ -57,6 +57,6 @@
 		axis = "0 1 0"
 		Lxx="21.53"
-		Lxy="0"
-		Lxz="0"
+		Lxy="0.0"
+		Lxz="0.0"
 		Lyy="10.896"
 		Lyz="0.14287"
@@ -70,7 +70,7 @@
 		upper_limit = "${radians(15)}"
 		velocity_limit = "300000.0"
-		joint_X = "0"
+		joint_X = "0.0"
 		joint_Y = "3.75000000"
-		joint_Z = "0"
+		joint_Z = "0.0"
 	/>
 	<!--Arm 3-->
@@ -97,6 +97,6 @@
 		velocity_limit = "300000.0"
 		joint_X = "18.00000000"
-		joint_Y = "0"
-		joint_Z = "0"
+		joint_Y = "0.0"
+		joint_Z = "0.0"
 	/>
 	<!--Arm 4-->
@@ -123,6 +123,6 @@
 		velocity_limit = "300000.0"
 		joint_X = "4.48622047"
-		joint_Y = "0"
-		joint_Z = "0"
+		joint_Y = "0.0"
+		joint_Z = "0.0"
 	/>
 	<!--Arm 5-->
@@ -149,6 +149,6 @@
 		velocity_limit = "300000.0"
 		joint_X = "17.25000000"
-		joint_Y = "0"
-		joint_Z = "0"
+		joint_Y = "0.0"
+		joint_Z = "0.0"
 	/>
 	<!--Arm 6-->
@@ -175,6 +175,6 @@
 		velocity_limit = "300000.0"
 		joint_X = "2.98622047"
-		joint_Y = "0"
-		joint_Z = "0"
+		joint_Y = "0.0"
+		joint_Z = "0.0"
 	/>
 	<!--Arm 7-->

Commit message: fixes

File: src/arm_control_moveit_config/config/robot_arm.ros2_control.xacro (robot description, xacro)
@@ -3,5 +3,5 @@
     <xacro:macro name="robot_arm_ros2_control" params="name initial_positions_file">
         <xacro:property name="initial_positions" value="${load_yaml(initial_positions_file)['initial_positions']}"/>
-  <ros2_control name="GazeboSystem" type="system">
+  <!-- <ros2_control name="GazeboSystem" type="system">
     <hardware>
       <plugin>gazebo_ros2_control/GazeboSystem</plugin>
@@ -43,7 +43,7 @@
       </state_interface>
     </joint>
-  </ros2_control>
-  <!-- <ros2_control name="yurs_motor" type="actuator"> -->
-        <!-- <hardware>
+  </ros2_control> -->
+  <ros2_control name="yurs_motor" type="actuator">
+        <hardware>
           <plugin>yurs_hardware/yurs_motor</plugin>
           <param name="can_interface">can0</param>
@@ -72,10 +72,10 @@
           <param name="device_id">11</param>
           <param name="counts_per_rev">1512</param>
-        </joint> -->
+        </joint>
         <!-- <joint name="arm_j7">
           <param name="device_id">12</param>
           <param name="counts_per_rev">1512</param>
         </joint> -->
-	<!-- </ros2_control> -->
+	</ros2_control>
     </xacro:macro>
 </robot>

File: src/arm_control_moveit_config/config/robot_arm.urdf.xacro (robot description, xacro)
@@ -6,4 +6,4 @@
     <!-- Import control_xacro -->
     <xacro:include filename="robot_arm.ros2_control.xacro" />
-    <xacro:robot_arm_ros2_control name="GazeboSystem" initial_positions_file="$(arg initial_positions_file)"/>
+    <xacro:robot_arm_ros2_control name="yurs_motor" initial_positions_file="$(arg initial_positions_file)"/>
 </robot>
