Commit message: arm control progress

File: src/my_bot/description/macros.xacro (robot description, xacro)
@@ -1,5 +1,4 @@
 <?xml version="1.0"?>
 <robot xmlns:xacro="http://www.ros.org/wiki/xacro"  >
-    <!-- <xacro:include filename="robot_core.xacro"/> -->
     <!--ROS2_CONTROL MACROS-->
     <!--Joint Creator-->
@@ -13,4 +12,13 @@
             <state_interface name="position"/>
         </joint>
+    </xacro:macro>
+    <xacro:macro name="arm_joint_creator" params="name">
+            <joint name="${name}">
+                <command_interface name="position"/>
+                <state_interface name="position">
+                    <param name="initial_value">0.0</param>
+                </state_interface>
+                <state_interface name="velocity"/>
+            </joint>
     </xacro:macro>
     <!--ROBOT_CORE MACROS-->
@@ -112,5 +120,5 @@
             <origin xyz="0 0 0" rpy="${radians(90)} 0 0"/>
             <geometry>
-                <mesh filename="file://$(find my_bot)/description/mesh/${file}.STL"/>
+                <mesh filename="file://$(find my_bot)/description/mesh/${file}.STL" />
             </geometry>
             <material name="white"/>
@@ -118,5 +126,5 @@
     </xacro:macro>
     <!-- Units: lb, in, lb*in^2 -->
-    <xacro:macro name="sw_inertial" params="m X Y Z Lxx Lxy Lxz Lyy Lyz Lzz">
+    <xacro:macro name="sw_inertial" params="m X Y Z Lxx Lxy Lxz Lyy Lyz Lzz file">
         <inertial>
             <mass value="${m*lbtokg}"/>
@@ -127,4 +135,10 @@
                 izz="${Lyy*lbsqintokgsqm}"/>
         </inertial>
+        <collision>
+            <xacro:sw_origin x="${X}" y="${Y}" z="${Z}"/>
+            <geometry>
+                <mesh filename="file://$(find my_bot)/description/mesh/${file}.STL" />
+            </geometry>
+        </collision>
     </xacro:macro>
 </robot>

File: src/my_bot/description/robot.urdf.xacro (robot description, xacro)
@@ -1,8 +1,7 @@
 <?xml version="1.0"?>
 <robot xmlns:xacro="http://www.ros.org/wiki/xacro"  name="robot">
-    <!-- <xacro:include filename="robot_core.xacro"/>
-    <xacro:include filename="ros2_control.xacro"/> -->
-    <xacro:include filename="arm.xacro"/>
+    <xacro:include filename="robot_core.xacro"/>
+    <xacro:include filename="ros2_control.xacro"/>
     <!-- <xacro:include filename="camera.xacro"/> -->
-    <!-- <xacro:include filename="depth_camera.xacro"/> -->
+    <xacro:include filename="depth_camera.xacro"/>
 </robot>

File: src/my_bot/description/robot_core.xacro (robot description, xacro)
@@ -6,6 +6,5 @@
     <xacro:property name="wheel_length" value="0.05" />
     <xacro:property name="chassis_origin" value="0 0 0.1" />
-    <!-- <xacro:include filename="inertial_macros.xacro"/> -->
-    <!-- <material name="white">
+    <material name="white">
         <color rgba="1 1 1 1"/>
     </material>
@@ -18,5 +17,5 @@
     <material name="black">
         <color rgba="0 0 0 1"/>
-    </material> -->
+    </material>
     <!-- WHEELS -->
     <!--With Encoders-->
@@ -30,12 +29,4 @@
     <!--BASE LINK-->
     <link name="base_link">
-    </link>
-    <!--BASE_FOOTPRINT LINK-->
-    <joint name ="base_footprint_joint" type="fixed">
-        <parent link="base_link"/>
-        <child link="base_footprint"/>
-        <origin xyz ="0 0 0" rpy="0 0 0"/>
-    </joint>
-    <link name ="base_footprint">
     </link>
     <!--CHASSIS LINK-->
@@ -68,36 +59,3 @@
         <mu2 value="0.001"/>
     </gazebo>
-    <!--IMU Sensor-->
-    <link name="imu">
-        <sensor name="my_imu" type="imu">
-            <always_on>true</always_on>
-            <!--Publish at 30 hz-->
-            <update_rate>30</update_rate>
-            <plugin name="my_imu_plugin" filename="libgazebo_ros_imu_sensor.so">
-                <ros>
-                    <!--Will publish to /imu/data-->
-                    <namespace>/imu</namespace>
-                    <remapping>~/out:=data</remapping>
-                </ros>
-                <!--frame_name ommited, will be "my_link"-->
-            </plugin>
-        </sensor>
-    </link>
-    <link name ="imu_sensor">
-    </link>
-    <gazebo reference="imu_sensor">
-        <sensor name="my_imu" type="imu">
-            <always_on>true</always_on>
-            <!--Publish at 30 hz-->
-            <update_rate>30</update_rate>
-            <plugin name="my_imu_plugin" filename="libgazebo_ros_imu_sensor.so">
-                <ros>
-                    <!--Will publish to /imu/data-->
-                    <namespace>/imu</namespace>
-                    <remapping>~/out:=data</remapping>
-                </ros>
-                <!--frame_name ommited, will be "my_link"-->
-            </plugin>
-        </sensor>
-    </gazebo>
 </robot>

Commit message: Deleted ambigous move it set up assistant and created a new moveit config dedicated for hardware launching

File: src/my_bot/description/macros.xacro (robot description, xacro)
@@ -163,5 +163,4 @@
                     izz="${Lyy*lbsqintokgsqm}"/>
             </inertial>
-<!--
             <collision>
                 <origin rpy="${radians(90)} 0 0" xyz="0 0 0"/>
@@ -169,5 +168,5 @@
                     <mesh filename="file://$(find my_bot)/description/mesh/${file}.STL" />
                 </geometry>
-            </collision> -->
+            </collision>
         </link>
         <joint name="arm_j${component_number}" type="${type}">
