Commit message: specification: modificating launch files

File: src/my_bot/description/arm.urdf (robot description, URDF)
Before this commit: robot robot_arm, 8 links, 7 joints
Joints:
- joint arm_j2: axis 0 1 0 -> 0 -1 0; limit lower=-2.356194490192345 upper=0.2617993877991494 effort=125000.0 velocity=300000.0 -> lower=-0.2617993877991494 upper=2.356194490192345 effort=125000.0 velocity=300000.0
